File: Slave/DifferentialEncoderSlave.kicad_pcb (KiCad board)
At the start: 4 copper layers, 52.5 x 24.8 mm, 32 parts, among them J1 Main, J2 Debug, J3 Thermistor, U1 ADM4852, U2 STM32G4A1KEU4, U3 LP5907MFX-3.3, U4 MA730

Commit message: Solomon redux
Parts:
- removed R1: 120, Resistor_SMD:R_0402_1005Metric
- removed TP5, TP6: TestPoint, ODrive_KiCad:TestPoint_Pad_D1.0mm
- added C10: 100nF, Capacitor_SMD:C_0402_1005Metric, F.Cu at (123.1, 75.0)
- added C11: 4.7uF, Capacitor_SMD:C_0603_1608Metric, F.Cu at (133.1, 68.9)
- added C12: 100nF, Capacitor_SMD:C_0402_1005Metric, F.Cu at (127.8, 77.4)
- added C13: 100nF, Capacitor_SMD:C_0402_1005Metric, F.Cu at (132.5, 70.2)
- added C14: 10pF, Capacitor_SMD:C_0402_1005Metric, F.Cu at (128.2, 67.6)
- added C15: 10pF, Capacitor_SMD:C_0402_1005Metric, F.Cu at (132.1, 67.3)
- added C16: 100nF, Capacitor_SMD:C_0402_1005Metric, F.Cu at (126.5, 75.0)
- added C8: 1uF, Capacitor_SMD:C_0402_1005Metric, F.Cu at (120.0, 67.2)
- added C9: 100nF, Capacitor_SMD:C_0402_1005Metric, F.Cu at (121.0, 67.2)
- added D1: SMF5.0CA, Diode_SMD:D_SOD-123F, F.Cu at (112.2, 74.3)
- added D2: LTST-C190KGKT, LED_SMD:LED_0603_1608Metric, F.Cu at (116.9, 65.3)
- added D3: LTST-C19HE1WT, LED_SMD:LED_LiteOn_LTST-C19HE1WT, F.Cu at (110.2, 84.3)
- added D4: SM712, Package_TO_SOT_SMD:SOT-23, F.Cu at (116.4, 73.5)
- added G***: LOGO, LOGO, B.Cu at (121.7, 79.7)
- added G***: LOGO, LOGO, B.Cu at (121.9, 84.0)
- added R3: 120, Resistor_SMD:R_0805_2012Metric, F.Cu at (119.1, 73.3)
- added R5: 1k, Resistor_SMD:R_0402_1005Metric, F.Cu at (118.9, 65.2)
- added R6: 10k, Resistor_SMD:R_0402_1005Metric, F.Cu at (133.8, 72.2)
- added R7: 600, Resistor_SMD:R_0402_1005Metric, F.Cu at (108.8, 80.1)
- added R8: 220, Resistor_SMD:R_0402_1005Metric, F.Cu at (109.8, 80.1)
- added R9: 220, Resistor_SMD:R_0402_1005Metric, F.Cu at (110.7, 80.1)
- added Y1: XRCGB16M000FXN00R0, Crystal:Crystal_SMD_2016-4Pin_2.0x1.6mm, F.Cu at (130.2, 67.5)
- C1: value 100nF -> 22uF; footprint Capacitor_SMD:C_0402_1005Metric -> Capacitor_SMD:C_0805_2012Metric
- C2, C4: value 100nF -> 1u
- H1, H2, H3, H4: footprint MountingHole:MountingHole_3mm -> mag-encoder:MountingHole_3.1mm_Pad_Via
- J2: value Debug -> PROG; footprint Connector:Tag-Connect_TC2030-IDC-NL_2x03_P1.27mm_Vertical -> Connector:Tag-Connect_TC2050-IDC-NL_2x05_P1.27mm_Vertical_with_bottom_clip
- R2: value 4.7k -> 3.3k/1%
- TP1, TP10, TP11, TP12, TP2, TP3, TP4, TP7, TP8, TP9: footprint ODrive_KiCad:TestPoint_Pad_D1.0mm -> TestPoint:TestPoint_Pad_1.0x1.0mm
- U4: value MA730 -> MA732
- moved J2 20.3 mm to (130.5, 63.2), turned to 0 degrees
- moved TP2 16.3 mm to (128.5, 78.7)
- moved TP3 16.2 mm to (130.0, 78.7)
- moved C1 14.4 mm to (112.3, 72.1)
- moved TP4 13.8 mm to (131.6, 78.7)
- moved TP1 12.1 mm to (135.3, 72.7)
- moved C2 11.1 mm to (115.2, 69.3), turned to -90 degrees
- moved U2 9.96 mm to (130.1, 73.8), turned to -90 degrees
- moved TP7 6.80 mm to (124.8, 70.1), turned to 90 degrees
- moved TP12 6.76 mm to (121.1, 72.2)
- moved TP11 6.44 mm to (121.1, 74.2)
- moved TP10 6.17 mm to (124.8, 68.6), turned to 90 degrees
- moved C4 6.07 mm to (120.3, 69.9)
- moved TP9 6.05 mm to (123.3, 70.1)
- moved TP8 3.12 mm to (124.8, 67.1)
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Connections:
- C1 pad 1: GNDD -> +5V
- C1 pad 2: +5V -> GND
- C2 pad 1: GNDD -> +5V
- C2 pad 2: +3V3 -> GND
- C3 pad 1: /~{RESET} -> /nRST
- C3 pad 2: GNDD -> GND
- C4 pad 1: GNDD -> +3V3
- C4 pad 2: +3V3 -> GND
- C5 pad 2: GNDD -> GND
- C6 pad 2: GNDD -> GND
- C7 pad 2: GNDD -> GND
- J1 pad 4: GNDD -> GND
- J1 pad SH: GNDD -> GND
- J2 pad 1: +5V -> +3V3
- J2 pad 2: /~{RESET} -> /SWO
- J2 pad 3: /SWCLK -> /SWDIO
- J2 pad 4: /SWDIO -> /USART2_TX
- J2 pad 5: GNDD -> GND
- J2 pad 6: GNDD -> GND
- J3 pad 2: GNDD -> GND
- J3 pad SH: GNDD -> GND
- TP4 pad 1: /USART2_DE -> /USART1_DE
- U1 pad 1: /USART2_RX -> /USART1_RX
- U1 pad 2: /USART2_DE -> /USART1_DE
- U1 pad 3: /USART2_DE -> /USART1_DE
- U1 pad 4: /USART2_TX -> /USART1_TX
- U1 pad 5: GNDD -> GND
- U2 pad 14: GNDD -> GND
- U2 pad 16: GNDD -> GND
- U2 pad 2: unconnected-(U2-Pad2) -> Net-(C15-Pad1)
- U2 pad 21: /USB_DN -> unconnected-(U2-Pad21)
- U2 pad 22: /USB_DP -> /USART1_DE
- U2 pad 26: /USART2_TX -> /SWO
- U2 pad 27: /USART2_RX -> /LED_R
- U2 pad 28: /I2S3_SD -> /LED_G
- U2 pad 3: unconnected-(U2-Pad3) -> Net-(C14-Pad2)
- U2 pad 30: unconnected-(U2-Pad30) -> /LED_B
- U2 pad 32: GNDD -> GND
- U2 pad 33: GNDD -> GND
- U2 pad 4: /~{RESET} -> /nRST
- U2 pad 6: /USART2_DE -> unconnected-(U2-Pad6)
- U2 pad 7: unconnected-(U2-Pad7) -> /USART2_TX
- U2 pad 8: unconnected-(U2-Pad8) -> /USART2_RX
- U3 pad 2: GNDD -> GND
- U4 pad 10: GNDD -> GND
- U4 pad 17: GNDD -> GND
- U4 pad 8: GNDD -> GND
Routing:
- net GNDD: track 61.3 -> 0.00 mm, vias 9 -> 0
- net /LED_B: track 0.00 -> 36.8 mm, vias 0 -> 2
- net /LED_G: track 0.00 -> 36.5 mm, vias 0 -> 2
- net /LED_R: track 0.00 -> 36.4 mm, vias 0 -> 2
- net +3V3: track 17.1 -> 46.9 mm, vias 3 -> 6
- net /~{RESET}: track 29.3 -> 0.00 mm, vias 2 -> 0
- net +5V: track 42.1 -> 59.8 mm, vias 3 -> 7
- net /SWO: track 0.00 -> 16.8 mm, vias 0 -> 2
- net /USART2_DE: track 15.4 -> 0.00 mm, vias 2 -> 0
- net /USART1_DE: track 0.00 -> 13.9 mm, vias 0 -> 2
- net /nRST: track 0.00 -> 11.8 mm, vias 0 -> 2
- net /USART1_TX: track 1.96 -> 12.7 mm, vias 0 -> 2
- net GND: track 0.00 -> 10.5 mm, vias 0 -> 171
- net /USART1_RX: track 1.45 -> 11.1 mm, vias 0 -> 2
- net /SWCLK: track 10.4 -> 19.7 mm
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- added copper zone on B.Cu, net GND
- added copper zone on F.Cu, net GND
- added copper zone on In1.Cu, net GND
- added copper zone on In2.Cu, net GND
- removed copper zone on In1.Cu, net +3V3
- removed copper zone on B.Cu, net +5V
- removed copper zone on F.Cu, net GNDD
- removed copper zone on In2.Cu, net GNDD
Other:
- outline, holes or cut-outs redrawn
- board text removed: "Keepout"
